File: ModuleNFC/ModuleNFC.kicad_pcb (KiCad board)
At the start: 2 copper layers, 48.8 x 38.8 mm, 45 parts, among them J1 Conn_01x10_Male, J2 Conn_01x04_Male, J3 Conn_01x08_Male, J4 Conn_Coaxial, Q1 2N7002DM, SW1 SW_DIP_x02, U1 PN5321A3HN_C1xx, Y1 27.12MHz

Commit message: Second revision of PCB and schematic, first change
Parts:
- moved D1 4.11 mm to (142.8, 107.1)
- moved Q1 3.04 mm to (137.6, 104.3)
- moved J2 3.03 mm to (133.8, 106.3)
- moved FID1 3.03 mm to (131.0, 118.6)
- moved R4 2.89 mm to (137.4, 100.8)
- moved R3 2.82 mm to (141.4, 104.4), turned to 90 degrees
- moved R5 2.75 mm to (137.6, 107.8)
- moved H2 2.26 mm to (132.3, 86.5)
Routing:
- net +3V3: track 46.1 -> 38.1 mm
- net /MOSI_SDA_TX: track 41.6 -> 35.4 mm
- net /NSS_SCL_RX: track 33.5 -> 30.2 mm
- net /SCK: track 23.8 -> 21.1 mm
- net /MISO: track 22.1 -> 19.5 mm
- net /RSTOUTN: track 31.5 -> 29.5 mm
- net /IRQ: track 16.1 -> 14.7 mm
- net Net-(D1-Pad2): track 2.08 -> 3.34 mm
Other:
- board size 48.8 x 38.8 mm -> 46.3 x 38.8 mm
- net class Default: clearance 0.2 -> 0.25
- rule trace_clearance: 0.2 -> 0.25
- board text added: "* El ancho de pista mínimo es: 0.25 mm * Se utilizo las capacidades de fabricación nacional (Mayer). * La capacidad de Mayer planteada para este módulo fue 10 mils * La grilla utilizada para acomodar componente cómo primera aproximación fue 1mm * La grilla utilizada para routear las pistas fue 0.1mm * El módelo 3D de Q1 utilizado es el SOT-23-6.wrl, este no es el encapsulado del componente pero e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"
- board text added: "Module NFC"
- board text removed: "* Las restricciones para el ancho de las pistas son los utilizados por fabricantes de industria nacional. * Se utilizo las capacidades de fabricación nacional (Mayer). * La capacidad de Mayer planteada para este módulo fue 10 mils * La grilla utilizada para acomodar componente cómo primera aproximación fue 1mm * La grilla utilizada para routear las pistas fue 0.1mm * El módelo 3D de Q1 utilizado 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"

Commit message: Correction final v1
Parts:
- added LOGO1: Logo_Open_Hardware_Small, Symbol:OSHW-Logo2_7.3x6mm_SilkScreen, F.Cu at (164.0, 86.0)
- added LOGO2: Logo_Open_Hardware_Small, Symbol:KiCad-Logo2_5mm_Copper, B.Cu at (136.5, 91.5)
- moved FID2 1.13 mm to (172.2, 118.0)
- moved FID1 0.60 mm to (131.0, 118.0)
- moved FID3 0.60 mm to (172.2, 85.0)
Other:
- board size 46.3 x 38.8 mm -> 47 x 39 mm
- board text added: "* Board dimension 47x39mm * Minimum (Mayer 10 mils) * Grid: 1mm, 0.1mm * Vias: 0.8/0.4 mm * Clearance: 0.25 mm * Track 0.25 mm * Surface finish: HASL * Thickness: 1.6 mm * El módelo 3D de Q1 utilizado es el SOT-23-6.wrl, este no es el encapsulado del componente pero es el que más se asemeja a las especificáciones de lo que se encontro en Internet. * Queda pendiente el análisis de impedancia en la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"
- board text added: "IND. ARG"
- board text removed: "* El ancho de pista mínimo es: 0.25 mm * Se utilizo las capacidades de fabricación nacional (Mayer). * La capacidad de Mayer planteada para este módulo fue 10 mils * La grilla utilizada para acomodar componente cómo primera aproximación fue 1mm * La grilla utilizada para routear las pistas fue 0.1mm * El módelo 3D de Q1 utilizado es el SOT-23-6.wrl, este no es el encapsulado del componente pero e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"
- board text removed: "KiCad E.D.A IND. ARG"
