File: ModuleNFC/ModuleNFC.kicad_pcb (KiCad board)
At the start: 2 copper layers, 47 x 39 mm, 47 parts, among them J1 Conn_01x10_Male, J2 Conn_01x04_Male, J3 Conn_01x08_Male, J4 Conn_Coaxial, Q1 2N7002DM, SW1 SW_DIP_x02, U1 PN5321A3HN_C1xx, Y1 27.12MHz

Commit message: Last version of correction
Parts:
- moved LOGO2 2.50 mm to (139.0, 91.5)
Other:
- board text added: "* Board dimension 47x39mm * Minimum (Mayer 10 mils) * Grid: 1mm, 0.5mm, 0.1mm * Vias: 0.8/0.4 mm * Clearance: 0.25 mm * Track 0.25 mm * Surface finish: HASL * Thickness: 1.6 mm * El módelo 3D de Q1 utilizado es el SOT-23-6.wrl, este no es el encapsulado del componente pero es el que más se asemeja a las especificáciones de lo que se encontro en Internet. * Queda pendiente el análisis de impedanci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"
- board text removed: "* Board dimension 47x39mm * Minimum (Mayer 10 mils) * Grid: 1mm, 0.1mm * Vias: 0.8/0.4 mm * Clearance: 0.25 mm * Track 0.25 mm * Surface finish: HASL * Thickness: 1.6 mm * El módelo 3D de Q1 utilizado es el SOT-23-6.wrl, este no es el encapsulado del componente pero es el que más se asemeja a las especificáciones de lo que se encontro en Internet. * Queda pendiente el análisis de impedancia en la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"
