File: ModuleNFC/ModuleNFC.sch (KiCad schematic (older format))
At the start: 46 parts, among them J1 Conn_01x10_Male, J2 Conn_01x04_Male, J3 Conn_01x08_Male, J4 Conn_Coaxial, Q1 2N7002DM, SW1 SW_DIP_x02, U1 PN5321A3HN_C1xx, Y1 27.12MHz

Commit message: Last version of correction
Parts:
- added LOGO2: Logo_Open_Hardware_Small, Symbol:KiCad-Logo2_5mm_Copper, symbol Graphic:Logo_Open_Hardware_Small
Changed lines of the file:
@@
+	1    0    0    -1
+$EndComp
+$Comp
+L Graphic:Logo_Open_Hardware_Small LOGO2
+U 1 1 5FB331B0
+P 9425 3050
+F 0 "LOGO2" H 9425 3325 50  0001 C CNN
+F 1 "Logo_Open_Hardware_Small" H 9425 2825 50  0001 C CNN
+F 2 "Symbol:KiCad-Logo2_5mm_Copper" H 9425 3050 50  0001 C CNN
+F 3 "~" H 9425 3050 50  0001 C CNN
+	1    9425 3050
 	1    0    0    -1
 $EndComp
